File: Hardware/core/_autosave-bootstrap.kicad_sch (KiCad schematic)
At the start: 25 parts

Commit message: osc pll pmuio
Parts:
- added R?: 10K, Resistor_SMD:R_0402_1005Metric, symbol Device:R
Connections:
- net BC_PMUIO1_VDD: now also R?.2; no longer U?.Y8 (FLASH_VOL_SEL/GPIO0_B3_d)
- new net: R?.1, U?.Y8 (FLASH_VOL_SEL/GPIO0_B3_d)
Changed lines of the file:
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@@
     (stroke (width 0) (type solid) (color 0 0 0 0))
   )
-  (wire (pts (xy 189.23 102.87) (xy 242.57 102.87))
+  (wire (pts (xy 189.23 102.87) (xy 204.47 102.87))
     (stroke (width 0) (type solid) (color 0 0 0 0))
   )
@@
   )
   (wire (pts (xy 212.09 73.66) (xy 242.57 73.66))
+    (stroke (width 0) (type solid) (color 0 0 0 0))
+  )
+  (wire (pts (xy 212.09 102.87) (xy 242.57 102.87))
     (stroke (width 0) (type solid) (color 0 0 0 0))
   )
@@
     )
   )
-  (global_label "BC_PMUIO1_VDD" (shape input) (at 242.57 102.87 0) (fields_autoplaced)
+  (global_label "BC_PMUIO1_VDD" (shape output) (at 242.57 102.87 0) (fields_autoplaced)
     (effects (font (size 1.27 1.27)) (justify left))
     (property "Intersheet References" "${INTERSHEET_REFS}" (id 0) (at 260.2836 102.7906 0)
@@
       (effects (font (size 1.27 1.27)) hide)
     )
+    (pin "1")
+    (pin "2")
+  )
+  (symbol (lib_id "Device:R") (at 208.28 102.87 90) (unit 1)
+    (in_bom yes) (on_board yes) (fields_autoplaced)
+    (property "Reference" "R?" (id 0) (at 208.28 97.79 90))
+    (property "Value" "10K" (id 1) (at 208.28 100.33 90))
+    (property "Footprint" "Resistor_SMD:R_0402_1005Metric" (id 2) (at 208.28 104.648 90)
+      (effects (font (size 1.27 1.27)) hide)
+    )
+    (property "Datasheet" "~" (id 3) (at 208.28 102.87 0)
+      (effects (font (size 1.27 1.27)) hide)
+    )
+    (property "Value2" "5%" (id 4) (at 208.28 102.87 90)
+      (effects (font (size 1.27 1.27)) hide)
+    )
