File: Hardware/core/audio.kicad_sch (KiCad schematic)
At the start: 1 part

Commit message: test
Parts:
- removed U?: RK809, berryflight:QFN-68_EP_7x7_Pitch0.35mm, symbol berryflight:RK809
Changed lines of the file:
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@@
     )
   )
-  (symbol (lib_id "berryflight:RK809") (at 83.82 45.72 0) (unit 3)
-    (in_bom yes) (on_board yes) (fields_autoplaced)
-    (property "Reference" "U?" (id 0) (at 97.79 41.91 0))
-    (property "Value" "RK809" (id 1) (at 97.79 44.45 0))
-    (property "Footprint" "berryflight:QFN-68_EP_7x7_Pitch0.35mm" (id 2) (at 104.14 39.37 0)
-      (effects (font (size 1.27 1.27)) hide)
-    )
-    (property "Datasheet" "" (id 3) (at 83.82 45.72 0)
-      (effects (font (size 1.27 1.27)) hide)
-    )
-    (pin "14")
-    (pin "15")
-    (pin "16")
-    (pin "17")
-    (pin "18")
-    (pin "19")
-    (pin "32")
-    (pin "33")
-    (pin "34")
-    (pin "35")
-    (pin "36")
-    (pin "37")
-    (pin "38")
-    (pin "39")
-    (pin "40")
-    (pin "41")
-    (pin "42")
-    (pin "43")
-    (pin "44")
-    (pin "48")
-  )
 )
