File: Hardware/core/bootstrap.kicad_sch (KiCad schematic)
At the start: 26 parts

Commit message: no ram yet
Parts:
- U1: renamed from U?; footprint berryflight: RV1126 -> berryflight:RV1126
- Y1: renamed from Y?; footprint (none) -> Oscillator:Oscillator_SMD_Abracon_ASE-4Pin_3.2x2.5mm
- gave numbers to parts that had none: 24
