File: Hardware/core/core.kicad_pcb (KiCad board)
At the start: 0 parts

Commit message: no ram yet
Parts:
- added C1: C100nF, Capacitor_SMD:C_0201_0603Metric, F.Cu at (116.3, 74.7)
- added C10: C1uF, Capacitor_SMD:C_0402_1005Metric, F.Cu at (239.9, 41.9)
- added C11: C1uF, Capacitor_SMD:C_0402_1005Metric, F.Cu at (186.2, 158.6)
- added C12: C1uF, Capacitor_SMD:C_0402_1005Metric, F.Cu at (186.2, 153.4)
- added C13: C100nF, Capacitor_SMD:C_0201_0603Metric, F.Cu at (225.6, 53.0)
- added C14: C10uF, Capacitor_SMD:C_0402_1005Metric, F.Cu at (165.3, 144.2)
- added C15: C10uF, Capacitor_SMD:C_0402_1005Metric, F.Cu at (165.3, 148.8)
- added C16: C1uF, Capacitor_SMD:C_0402_1005Metric, F.Cu at (186.2, 148.3)
- added C17: C100nF, Capacitor_SMD:C_0201_0603Metric, F.Cu at (128.5, 62.8)
- added C18: C10uF, Capacitor_SMD:C_0402_1005Metric, F.Cu at (165.3, 153.4)
- added C19: C100nF, Capacitor_SMD:C_0201_0603Metric, F.Cu at (128.5, 67.2)
- added C2: C100nF, Capacitor_SMD:C_0201_0603Metric, F.Cu at (110.9, 75.7)
- added C20: C1uF, Capacitor_SMD:C_0402_1005Metric, F.Cu at (186.2, 143.1)
- added C21: C1uF, Capacitor_SMD:C_0402_1005Metric, F.Cu at (109.9, 55.4)
- added C22: C10uF, Capacitor_SMD:C_0603_1608Metric, F.Cu at (159.8, 158.3)
- added C23: C10uF, Capacitor_SMD:C_0603_1608Metric, F.Cu at (171.9, 137.1)
- added C24: C10uF, Capacitor_SMD:C_0603_1608Metric, F.Cu at (154.4, 158.2)
- added C25: C10uF, Capacitor_SMD:C_0402_1005Metric, F.Cu at (170.4, 142.6)
- added C26: C10uF, Capacitor_SMD:C_0603_1608Metric, F.Cu at (149.1, 158.3)
- added C27: C10uF, Capacitor_SMD:C_0603_1608Metric, F.Cu at (143.6, 158.3)
- added C28: C22uF, Capacitor_SMD:C_0603_1608Metric, F.Cu at (103.9, 64.3)
- added C29: C22uF, Capacitor_SMD:C_0603_1608Metric, F.Cu at (103.7, 69.6)
- added C3: C100nF, Capacitor_SMD:C_0201_0603Metric, F.Cu at (110.9, 80.1)
- added C30: C22uF, Capacitor_SMD:C_0603_1608Metric, F.Cu at (103.7, 75.2)
- added C31: C22uF, Capacitor_SMD:C_0603_1608Metric, F.Cu at (110.4, 60.2)
- added C32: C10uF, Capacitor_SMD:C_0603_1608Metric, F.Cu at (110.4, 65.4)
- added C33: C22uF, Capacitor_SMD:C_0603_1608Metric, F.Cu at (110.2, 70.7)
- added C34: C22uF, Capacitor_SMD:C_0603_1608Metric, F.Cu at (122.4, 63.7)
- added C35: C1uF, Capacitor_SMD:C_0402_1005Metric, F.Cu at (166.9, 137.3)
- added C36: C100nF, Capacitor_SMD:C_0402_1005Metric, F.Cu at (213.0, 41.9)
- added C37: C1uF, Capacitor_SMD:C_0402_1005Metric, F.Cu at (212.1, 37.3)
- added C38: C1uF, Capacitor_SMD:C_0402_1005Metric, F.Cu at (218.5, 37.3)
- added C39: C1uF, Capacitor_SMD:C_0402_1005Metric, F.Cu at (235.4, 37.3)
- added C4: C10uF, Capacitor_SMD:C_0603_1608Metric, B.Cu at (170.8, 158.3)
- added C40: C1uF, Capacitor_SMD:C_0402_1005Metric, F.Cu at (237.6, 48.5)
- added C41: C1uF, Capacitor_SMD:C_0402_1005Metric, F.Cu at (127.6, 58.3)
- added C42: C10uF, Capacitor_SMD:C_0603_1608Metric, F.Cu at (116.9, 63.7)
- added C43: C22uF, Capacitor_SMD:C_0603_1608Metric, F.Cu at (116.9, 68.9)
- added C44: C1uF, Capacitor_SMD:C_0402_1005Metric, F.Cu at (116.4, 58.8)
- added C45: C1uF, Capacitor_SMD:C_0402_1005Metric, F.Cu at (121.9, 58.8)
- added C46: C1uF, Capacitor_SMD:C_0402_1005Metric, F.Cu at (211.3, 66.0)
- added C47: C1uF, Capacitor_SMD:C_0402_1005Metric, F.Cu at (211.3, 48.3)
- added C48: C1uF, Capacitor_SMD:C_0402_1005Metric, F.Cu at (235.4, 41.9)
- added C49: C1uF, Capacitor_SMD:C_0402_1005Metric, F.Cu at (103.4, 59.4)
- added C5: C100nF, Capacitor_SMD:C_0402_1005Metric, F.Cu at (219.5, 41.9)
- added C50: C1uF, Capacitor_SMD:C_0402_1005Metric, F.Cu at (143.1, 144.2)
- added C51: C1uF, Capacitor_SMD:C_0402_1005Metric, F.Cu at (143.1, 148.8)
- added C52: C1uF, Capacitor_SMD:C_0402_1005Metric, F.Cu at (143.1, 153.4)
- added C53: C1uF, Capacitor_SMD:C_0402_1005Metric, F.Cu at (148.6, 143.7)
- added C54: C1uF, Capacitor_SMD:C_0402_1005Metric, F.Cu at (148.6, 148.3)
- added C55: C22uF, Capacitor_SMD:C_0603_1608Metric, F.Cu at (181.6, 137.1)
- added C56: C15pF, Capacitor_SMD:C_0402_1005Metric, F.Cu at (83.3, 148.1)
- added C57: 1uF, Capacitor_SMD:C_0402_1005Metric, F.Cu at (93.4, 133.4)
- added C58: 1uF, Capacitor_SMD:C_0402_1005Metric, F.Cu at (99.8, 155.8)
- added C59: 100nF, Capacitor_SMD:C_0201_0603Metric, F.Cu at (88.8, 139.4)
- added C6: C100nF, Capacitor_SMD:C_0201_0603Metric, F.Cu at (104.4, 80.1)
- added C60: 100nF, Capacitor_SMD:C_0201_0603Metric, F.Cu at (90.9, 156.0)
- added C61: 100nF, Capacitor_SMD:C_0201_0603Metric, F.Cu at (77.7, 143.6)
- added C62: 100nF, Capacitor_SMD:C_0201_0603Metric, F.Cu at (83.2, 143.6)
- added C63: 100nF, Capacitor_SMD:C_0201_0603Metric, F.Cu at (88.8, 143.8)
- added C64: 100nF, Capacitor_SMD:C_0201_0603Metric, F.Cu at (88.8, 148.2)
- added C65: C15pF, Capacitor_SMD:C_0402_1005Metric, F.Cu at (77.8, 148.1)
- added C66: 100nF, Capacitor_SMD:C_0402_1005Metric, F.Cu at (85.5, 155.8)
- added C67: 10uF, Capacitor_SMD:C_0805_2012Metric, B.Cu at (114.2, 95.1)
- added C68: 1uF, Capacitor_SMD:C_0402_1005Metric, B.Cu at (128.0, 93.0)
- added C69: 10uF, Capacitor_SMD:C_0805_2012Metric, B.Cu at (97.3, 100.8)
- added C7: C100nF, Capacitor_SMD:C_0201_0603Metric, F.Cu at (232.1, 48.6)
- added C70: 10uF, Capacitor_SMD:C_0805_2012Metric, B.Cu at (103.2, 100.9)
- added C71: 100nF, Capacitor_SMD:C_0402_1005Metric, B.Cu at (111.1, 95.1)
- added C72: 100nF, Capacitor_SMD:C_0402_1005Metric, B.Cu at (128.9, 93.0)
- added C73: 10nF, Capacitor_SMD:C_0402_1005Metric, B.Cu at (96.6, 95.5)
- added C74: 10nF, Capacitor_SMD:C_0402_1005Metric, B.Cu at (102.4, 94.7)
- added C75: 100nF, Capacitor_SMD:C_0402_1005Metric, B.Cu at (112.1, 95.1)
- added C76: 100pF, Capacitor_SMD:C_0402_1005Metric, B.Cu at (96.6, 93.9)
- added C77: 100pF, Capacitor_SMD:C_0402_1005Metric, B.Cu at (102.4, 93.9)
- added C78: 1uF, Capacitor_SMD:C_0402_1005Metric, B.Cu at (125.7, 90.8)
- added C79: 22pF, Capacitor_SMD:C_0402_1005Metric, B.Cu at (110.2, 93.4)
- added C8: C100nF, Capacitor_SMD:C_0201_0603Metric, F.Cu at (225.6, 48.6)
- added C80: 22pF, Capacitor_SMD:C_0805_2012Metric, B.Cu at (111.2, 89.8)
- added C81: 22uF, Capacitor_SMD:C_0603_1608Metric, B.Cu at (97.0, 89.6)
- added C82: 22uF, Capacitor_SMD:C_0603_1608Metric, B.Cu at (105.7, 89.6)
- added C83: 10uF, Capacitor_SMD:C_0805_2012Metric, B.Cu at (114.4, 89.8)
- added C84: 100nF, Capacitor_SMD:C_0402_1005Metric, B.Cu at (96.6, 91.5)
- added C85: 100nF, Capacitor_SMD:C_0402_1005Metric, B.Cu at (102.4, 90.7)
- added C86: 100nF, Capacitor_SMD:C_0402_1005Metric, B.Cu at (111.1, 91.7)
- added C87: 22uF, Capacitor_SMD:C_0603_1608Metric, B.Cu at (99.9, 89.6)
- added C88: 22uF, Capacitor_SMD:C_0603_1608Metric, B.Cu at (102.9, 89.6)
- added C89: 100nF, Capacitor_SMD:C_0201_0603Metric, F.Cu at (81.9, 58.6)
- added C9: C10uF, Capacitor_SMD:C_0603_1608Metric, F.Cu at (165.3, 158.3)
- added C90: 100nF, Capacitor_SMD:C_0201_0603Metric, F.Cu at (62.7, 73.2)
- added C91: 100nF, Capacitor_SMD:C_0201_0603Metric, F.Cu at (65.6, 71.2)
- added C92: 1uF, Capacitor_SMD:C_0402_1005Metric, F.Cu at (63.0, 71.3)
- added C93: 1uF, Capacitor_SMD:C_0402_1005Metric, F.Cu at (60.0, 73.3)
- added C94: 1uF, Capacitor_SMD:C_0402_1005Metric, F.Cu at (82.1, 56.8)
- added C95: 10uF, Capacitor_SMD:C_0603_1608Metric, F.Cu at (56.6, 71.6)
- added D1: LED, LED_SMD:LED_0603_1608Metric, F.Cu at (139.8, 103.6)
- added L1: 470nH, Inductor_SMD:L_1008_2520Metric, F.Cu at (206.6, 41.4)
- added L2: 470nH, Inductor_SMD:L_1008_2520Metric, F.Cu at (206.2, 47.4)
- added L3: 470nH, Inductor_SMD:L_1008_2520Metric, F.Cu at (206.6, 53.4)
- added L4: 470nH, Inductor_SMD:L_1008_2520Metric, F.Cu at (206.6, 59.1)
- added L5: 470nH, Inductor_SMD:L_1008_2520Metric, F.Cu at (206.2, 65.1)
- added L6: 2.2uH, Inductor_SMD:L_1008_2520Metric, B.Cu at (99.4, 94.8)
- added L7: 2.2uH, Inductor_SMD:L_1008_2520Metric, B.Cu at (105.2, 94.8)
- added L8: 4.7uH, Inductor_SMD:L_TracoPower_TCK-047_5.2x5.8mm, B.Cu at (119.7, 93.8)
- added R1: 0.1R, Resistor_SMD:R_0603_1608Metric, F.Cu at (148.4, 153.2)
- added R10: 0.02R, Resistor_SMD:R_0805_2012Metric, F.Cu at (122.4, 72.0)
- added R11: 2.2K, Resistor_SMD:R_0402_1005Metric, F.Cu at (239.8, 37.2)
- added R12: 2.2K, Resistor_SMD:R_0402_1005Metric, F.Cu at (103.5, 55.0)
- added R13: 0R, Resistor_SMD:R_0402_1005Metric, F.Cu at (121.9, 54.6)
- added R14: 10K, Resistor_SMD:R_0402_1005Metric, F.Cu at (186.8, 132.7)
- added R15: 10K, Resistor_SMD:R_0402_1005Metric, F.Cu at (186.8, 137.3)
- added R16: 0R, Resistor_SMD:R_0402_1005Metric, F.Cu at (116.4, 54.7)
- added R17: 0R, Resistor_SMD:R_0402_1005Metric, F.Cu at (211.7, 59.6)
- added R18: 100K, Resistor_SMD:R_0402_1005Metric, F.Cu at (159.4, 153.4)
- added R19: 27K, Resistor_SMD:R_0402_1005Metric, F.Cu at (211.7, 53.9)
- added R2: 0.1R, Resistor_SMD:R_0603_1608Metric, F.Cu at (154.4, 143.9)
- added R20: 0.05R, Resistor_SMD:R_0603_1608Metric, F.Cu at (170.6, 148.0)
- added R21: 0.05R, Resistor_SMD:R_0603_1608Metric, F.Cu at (170.6, 153.2)
- added R22: 0.05R, Resistor_SMD:R_0603_1608Metric, F.Cu at (176.1, 142.8)
- added R23: 0.05R, Resistor_SMD:R_0603_1608Metric, F.Cu at (176.1, 148.0)
- added R24: 0.05R, Resistor_SMD:R_0603_1608Metric, F.Cu at (176.1, 153.2)
- added R25: 0.05R, Resistor_SMD:R_0603_1608Metric, F.Cu at (181.3, 142.8)
- added R26: 0.05R, Resistor_SMD:R_0603_1608Metric, F.Cu at (181.3, 148.0)
- added R27: 0.05R, Resistor_SMD:R_0603_1608Metric, F.Cu at (181.3, 153.2)
- added R28: 0.05R, Resistor_SMD:R_0603_1608Metric, F.Cu at (181.3, 158.3)
- added R29: 0.05R, Resistor_SMD:R_0603_1608Metric, F.Cu at (176.1, 158.3)
- added R3: 100R, Resistor_SMD:R_0402_1005Metric, F.Cu at (154.2, 148.4)
- added R30: 0.02R, Resistor_SMD:R_0805_2012Metric, F.Cu at (230.5, 41.4)
- added R31: 0.02R, Resistor_SMD:R_0805_2012Metric, F.Cu at (225.3, 41.4)
- added R32: 0,1R, Resistor_SMD:R_0603_1608Metric, F.Cu at (95.8, 150.4)
- added R33: 0,1R, Resistor_SMD:R_0603_1608Metric, F.Cu at (95.8, 155.6)
- added R34: 0,1R, Resistor_SMD:R_0603_1608Metric, F.Cu at (93.6, 138.3)
- added R35: 0,1R, Resistor_SMD:R_0603_1608Metric, F.Cu at (79.0, 138.8)
- added R36: 0,1R, Resistor_SMD:R_0603_1608Metric, F.Cu at (82.5, 140.8)
- added R37: 0,1R, Resistor_SMD:R_0603_1608Metric, F.Cu at (93.6, 143.4)
- added R38: 22R, Resistor_SMD:R_0402_1005Metric, F.Cu at (99.8, 150.7)
- added R39: 1M, Resistor_SMD:R_0402_1005Metric, F.Cu at (97.6, 133.9)
- added R4: 100R, Resistor_SMD:R_0402_1005Metric, F.Cu at (154.2, 153.1)
- added R40: 0R, Resistor_SMD:R_0402_1005Metric, F.Cu at (76.9, 133.9)
- added R41: 0R, Resistor_SMD:R_0402_1005Metric, F.Cu at (81.1, 133.9)
- added R42: 0R, Resistor_SMD:R_0402_1005Metric, F.Cu at (87.9, 134.9)
- added R43: 10K, Resistor_SMD:R_0402_1005Metric, F.Cu at (97.6, 143.7)
- added R44: 0R, Resistor_SMD:R_0402_1005Metric, F.Cu at (97.6, 138.5)
- added R45: 47K, Resistor_SMD:R_0402_1005Metric, B.Cu at (96.6, 97.9)
- added R46: 18K, Resistor_SMD:R_0402_1005Metric, B.Cu at (96.6, 97.1)
- added R47: 47K, Resistor_SMD:R_0402_1005Metric, B.Cu at (102.5, 97.9)
- added R48: 18K, Resistor_SMD:R_0402_1005Metric, B.Cu at (102.5, 96.3)
- added R49: 20K, Resistor_SMD:R_0402_1005Metric, B.Cu at (96.6, 99.5)
- added R5: 120K, Resistor_SMD:R_0402_1005Metric, F.Cu at (159.4, 144.1)
- added R50: 10K, Resistor_SMD:R_0402_1005Metric, B.Cu at (96.6, 98.7)
- added R51: 20K, Resistor_SMD:R_0402_1005Metric, B.Cu at (102.5, 98.7)
- added R52: 10K, Resistor_SMD:R_0402_1005Metric, B.Cu at (102.5, 99.5)
- added R53: 15K, Resistor_SMD:R_0402_1005Metric, B.Cu at (96.6, 96.3)
- added R54: 15K, Resistor_SMD:R_0402_1005Metric, B.Cu at (102.5, 95.5)
- added R55: 100K, Resistor_SMD:R_0402_1005Metric, B.Cu at (110.2, 95.1)
- added R56: 249K, Resistor_SMD:R_0402_1005Metric, B.Cu at (96.6, 94.7)
- added R57: 249K, Resistor_SMD:R_0402_1005Metric, B.Cu at (102.5, 97.1)
- added R58: 76.8K, Resistor_SMD:R_0402_1005Metric, B.Cu at (112.1, 93.4)
- added R59: 10K, Resistor_SMD:R_0402_1005Metric, B.Cu at (111.1, 93.4)
- added R6: 110K, Resistor_SMD:R_0402_1005Metric, F.Cu at (159.4, 148.8)
- added R60: 100R, Resistor_SMD:R_0402_1005Metric, B.Cu at (96.6, 92.3)
- added R61: 33K, Resistor_SMD:R_0402_1005Metric, B.Cu at (96.6, 93.1)
- added R62: 100R, Resistor_SMD:R_0402_1005Metric, B.Cu at (102.5, 93.1)
- added R63: 33K, Resistor_SMD:R_0402_1005Metric, B.Cu at (102.5, 92.3)
- added R64: 0.02R, Resistor_SMD:R_0805_2012Metric, B.Cu at (99.7, 92.7)
- added R65: 100K, Resistor_SMD:R_0402_1005Metric, B.Cu at (96.6, 90.7)
- added R66: 0.02R, Resistor_SMD:R_0805_2012Metric, B.Cu at (105.5, 92.7)
- added R67: 100K, Resistor_SMD:R_0402_1005Metric, B.Cu at (102.5, 91.5)
- added R68: 2K, Resistor_SMD:R_0402_1005Metric, B.Cu at (110.2, 91.7)
- added R69: 0.02R, Resistor_SMD:R_0805_2012Metric, B.Cu at (99.7, 91.0)
- added R7: 0.02R, Resistor_SMD:R_0805_2012Metric, F.Cu at (99.2, 84.8)
- added R70: 0.02R, Resistor_SMD:R_0805_2012Metric, B.Cu at (105.5, 91.1)
- added R71: DNP, Resistor_SMD:R_0402_1005Metric, B.Cu at (112.1, 91.7)
- added R72: 0.02R, Resistor_SMD:R_0805_2012Metric, B.Cu at (117.6, 89.8)
- added R73: 240R, Resistor_SMD:R_0402_1005Metric, F.Cu at (60.1, 71.3)
- added R8: 0.02R, Resistor_SMD:R_0805_2012Metric, F.Cu at (128.1, 72.0)
- added R9: 0.02R, Resistor_SMD:R_0805_2012Metric, F.Cu at (111.4, 84.8)
- added U1: RV1126, berryflight:RV1126, F.Cu at (67.8, 107.1)
- added U2: RK809, berryflight:QFN-68_EP_7x7_Pitch0.35mm, F.Cu at (238.3, 75.2)
- added U3: NCEPNA6M4-0808, berryflight:BGA-221, B.Cu at (69.5, 91.3)
- added U4: SY8089AAAC, Package_TO_SOT_SMD:SOT-23-5, B.Cu at (99.2, 98.0)
- added U5: SY8089AAAC, Package_TO_SOT_SMD:SOT-23-5, B.Cu at (104.9, 98.0)
- added U6: SY8113B, Package_TO_SOT_SMD:TSOT-23-6, B.Cu at (114.5, 92.4)
- added U7: SGM2203-5.0, Package_TO_SOT_SMD:SOT-23, B.Cu at (125.8, 93.0)
- added Y1: 24Mhz, Oscillator:Oscillator_SMD_Abracon_ASE-4Pin_3.2x2.5mm, F.Cu at (79.4, 153.8)
Routing:
- net /Storage and RAM/DQ1: track 0.00 -> 4.52 mm, vias 0 -> 2
- net /Storage and RAM/DQ0: track 0.00 -> 3.84 mm, vias 0 -> 2
- net /Storage and RAM/DQS0P: track 0.00 -> 2.67 mm, vias 0 -> 2
- net /Storage and RAM/DQS0N: track 0.00 -> 2.03 mm, vias 0 -> 2
- net /Storage and RAM/DM0: track 0.00 -> 2.02 mm, vias 0 -> 2
- net /Storage and RAM/DQ5: track 0.00 -> 2.01 mm, vias 0 -> 2
- net /Storage and RAM/DQ4: track 0.00 -> 2.00 mm, vias 0 -> 2
- net /Storage and RAM/DQS3P: vias 0 -> 1
- net /Storage and RAM/DQS3N: vias 0 -> 1
- net /Storage and RAM/DQS2P: vias 0 -> 1
- net /Storage and RAM/DQS2N: vias 0 -> 1
- net /Storage and RAM/DQS1P: vias 0 -> 1
- net /Storage and RAM/DQS1N: vias 0 -> 1
- net /Storage and RAM/DQ9: vias 0 -> 1
- net /Storage and RAM/DQ8: vias 0 -> 1
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Other:
- board outline added: 37 x 37 mm
- copper layers 0 -> 6
