File: Hardware/core/core.kicad_pcb (KiCad board)
At the start: 6 copper layers, 37 x 37 mm, 185 parts, among them U1 RV1126, U2 RK809, U3 NCEPNA6M4-0808, U4 SY8089AAAC, U5 SY8089AAAC, U6 SY8113B, U7 SGM2203-5.0, Y1 24Mhz

Commit message: byte0?
Parts:
- moved U3 4.28 mm to (68.1, 95.4), turned to -90 degrees
- moved U1 3.63 mm to (69.0, 110.6)
Connections:
- U3 pad H9: /Storage and RAM/DQS3N -> /Storage and RAM/DQS3P
- U3 pad J9: /Storage and RAM/DQS3P -> /Storage and RAM/DQS3N
- U3 pad M9: /Storage and RAM/DQS1N -> /Storage and RAM/DQS1P
- U3 pad N3: /Storage and RAM/CLKP -> /Storage and RAM/CLKN
- U3 pad N9: /Storage and RAM/DQS1P -> /Storage and RAM/DQS1N
- U3 pad P3: /Storage and RAM/CLKN -> /Storage and RAM/CLKP
- U3 pad R9: /Storage and RAM/DQS0P -> /Storage and RAM/DQS0N
- U3 pad T9: /Storage and RAM/DQS0N -> /Storage and RAM/DQS0P
- U3 pad W9: /Storage and RAM/DQS2P -> /Storage and RAM/DQS2N
- U3 pad Y9: /Storage and RAM/DQS2N -> /Storage and RAM/DQS2P
Routing:
- net /Storage and RAM/DQS0P: track 2.67 -> 15.9 mm, vias 2 -> 0
- net /Storage and RAM/DQS0N: track 2.03 -> 12.2 mm, vias 2 -> 0
- net /Storage and RAM/DQ2: track 0.00 -> 9.05 mm, vias 2 -> 0
- net /Storage and RAM/DQ7: track 0.00 -> 8.05 mm, vias 2 -> 0
- net /Storage and RAM/DQ3: track 0.00 -> 5.12 mm, vias 2 -> 0
- net /Storage and RAM/DQ0: track 3.84 -> 8.64 mm, vias 2 -> 0
- net /Storage and RAM/DQ6: track 0.00 -> 4.17 mm, vias 2 -> 0
- net /Storage and RAM/DM0: track 2.02 -> 5.57 mm, vias 2 -> 0
- net /Storage and RAM/DQ5: track 2.01 -> 5.40 mm, vias 2 -> 0
- net /Storage and RAM/DQ1: track 4.52 -> 6.57 mm, vias 2 -> 0
- net /Storage and RAM/DQ4: track 2.00 -> 3.02 mm, vias 2 -> 0
- net /Storage and RAM/DQS3P: vias 1 -> 0
- net /Storage and RAM/DQS3N: vias 1 -> 0
- net /Storage and RAM/DQS2P: vias 1 -> 0
- net /Storage and RAM/DQS2N: vias 1 -> 0
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