File: Hardware/core/core.kicad_pcb (KiCad board)
At the start: 6 copper layers, 37 x 37 mm, 185 parts, among them U1 RV1126, U2 RK809, U3 NCEPNA6M4-0808, U4 SY8089AAAC, U5 SY8089AAAC, U6 SY8113B, U7 SGM2203-5.0, Y1 24Mhz

Commit message: byte3 and address
Parts:
- moved U3 15.8 mm to (82.4, 102.0), turned to 180 degrees
Routing:
- net /Storage and RAM/DQS2N: track 0.00 -> 16.2 mm
- net /Storage and RAM/DQS2P: track 0.00 -> 12.7 mm
- net /Storage and RAM/A0: track 0.00 -> 12.0 mm
- net /Storage and RAM/A2: track 0.00 -> 11.5 mm
- net /Storage and RAM/A7: track 0.00 -> 10.2 mm
- net /Storage and RAM/A9: track 0.00 -> 10.2 mm
- net /Storage and RAM/DM2: track 0.00 -> 10.1 mm
- net /Storage and RAM/A3: track 0.00 -> 9.20 mm
- net /Storage and RAM/A6: track 0.00 -> 8.54 mm
- net /Storage and RAM/A8: track 0.00 -> 8.47 mm
- net /Storage and RAM/A5: track 0.00 -> 8.28 mm
- net /Storage and RAM/DQ19: track 0.00 -> 6.57 mm
- net /Storage and RAM/DQ21: track 0.00 -> 4.84 mm
- net /Storage and RAM/DQ18: track 0.00 -> 4.55 mm
- net /Storage and RAM/DM1: track 13.7 -> 9.85 mm
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
Commit message: ...
Parts:
- moved R55 47.6 mm to (149.8, 121.5), turned to 180 degrees
- moved C79 47.2 mm to (148.1, 121.5), turned to 0 degrees
- moved R68 46.9 mm to (146.3, 121.5), turned to 180 degrees
- moved C71 46.3 mm to (149.8, 120.6), turned to 180 degrees
- moved R59 45.9 mm to (148.1, 120.6), turned to 0 degrees
- moved C86 45.6 mm to (146.4, 120.6), turned to 180 degrees
- moved C80 45.3 mm to (144.5, 120.5), turned to -90 degrees
- moved C75 45.0 mm to (149.8, 119.6), turned to 180 degrees
- moved R58 44.5 mm to (148.1, 119.6), turned to 0 degrees
- moved R71 44.2 mm to (146.3, 119.6), turned to 180 degrees
- moved U1 42.8 mm to (111.7, 112.0)
- moved C67 42.1 mm to (149.8, 117.5), turned to -90 degrees
- moved U6 41.0 mm to (147.1, 117.2), turned to -90 degrees
- moved C83 40.8 mm to (144.5, 117.3), turned to -90 degrees
- moved R72 36.3 mm to (144.5, 114.1), turned to -90 degrees
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Connections:
- U1 pad L3: /Storage and RAM/DQS0N -> /Storage and RAM/DQ6
- U1 pad N3: /Storage and RAM/DM0 -> /Storage and RAM/MMC_D7
Routing:
- net /Storage and RAM/DQ6: track 4.27 -> 29.8 mm, vias 0 -> 4
- net /Storage and RAM/MMC_D7: track 10.9 -> 35.9 mm, vias 0 -> 4
- net /Storage and RAM/A9: track 10.2 -> 27.1 mm, vias 0 -> 2
- net /Storage and RAM/A8: track 8.47 -> 24.9 mm, vias 0 -> 2
- net /Storage and RAM/A7: track 10.2 -> 26.1 mm, vias 0 -> 2
- net /Storage and RAM/A6: track 8.54 -> 22.0 mm, vias 0 -> 2
- net /Storage and RAM/A5: track 8.28 -> 21.3 mm, vias 0 -> 2
- net /Storage and RAM/A4: track 2.45 -> 15.3 mm, vias 0 -> 1
- net /Storage and RAM/MMC_D2: track 6.79 -> 19.4 mm, vias 0 -> 2
- net /Storage and RAM/A1: track 2.15 -> 14.6 mm, vias 0 -> 1
- net /Storage and RAM/MMC_D6: track 6.36 -> 17.4 mm, vias 0 -> 2
- net /Storage and RAM/DQS0N: track 10.9 -> 0.00 mm
- net /Storage and RAM/DQ5: track 5.40 -> 15.3 mm, vias 0 -> 2
- net /Storage and RAM/DQ3: track 5.05 -> 14.4 mm, vias 0 -> 2
- net /Storage and RAM/DQ4: track 3.02 -> 12.2 mm, vias 0 -> 2
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