File: Hardware/core/core.kicad_sch (KiCad schematic)
At the start: 0 parts

Commit message: test
Other:
- added sheet more power supplys (more power.kicad_sch)
Changed lines of the file:
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@@
     (effects (font (size 3 3)) (justify left bottom))
   )
-  (sheet (at 30.48 90.17) (size 53.34 29.21) (fields_autoplaced)
+  (sheet (at 90.17 87.63) (size 53.34 29.21) (fields_autoplaced)
     (stroke (width 0.0006) (type solid) (color 0 0 0 0))
     (fill (color 0 0 0 0.0000))
-    (property "Sheet name" "Audio" (id 0) (at 30.48 89.5343 0)
+    (property "Sheet name" "Audio" (id 0) (at 90.17 86.9943 0)
       (effects (font (size 1.27 1.27)) (justify left bottom))
     )
-    (property "Sheet file" "audio.kicad_sch" (id 1) (at 30.48 119.8887 0)
+    (property "Sheet file" "audio.kicad_sch" (id 1) (at 90.17 117.3487 0)
       (effects (font (size 1.27 1.27)) (justify left top))
     )
@@
     )
     (property "Sheet file" "memory.kicad_sch" (id 1) (at 149.86 76.7087 0)
+      (effects (font (size 1.27 1.27)) (justify left top))
+    )
+  )
+  (sheet (at 30.48 87.63) (size 53.34 29.21) (fields_autoplaced)
+    (stroke (width 0.0006) (type solid) (color 0 0 0 0))
+    (fill (color 0 0 0 0.0000))
+    (property "Sheet name" "more power supplys" (id 0) (at 30.48 86.9943 0)
+      (effects (font (size 1.27 1.27)) (justify left bottom))
+    )
+    (property "Sheet file" "more power.kicad_sch" (id 1) (at 30.48 117.3487 0)
       (effects (font (size 1.27 1.27)) (justify left top))
     )
@@
     (path "/a74c9d3b-864a-43d5-bde6-cbf00bb39165/" (page "5"))
     (path "/e25c5f3e-57b5-4d7a-a8af-98b1826cae36/" (page "6"))
+    (path "/2b4337a7-31ba-4b62-90e4-5bec465ff16f/" (page "7"))
   )
   (symbol_instances
@@
       (reference "R?") (unit 1) (value "0,1R") (footprint "Resistor_SMD:R_0603_1608Metric")
     )
+    (path "/a74c9d3b-864a-43d5-bde6-cbf00bb39165/fcf47248-2ab2-4874-8e1b-f981cb0c8c68"
+      (reference "R?") (unit 1) (value "10K") (footprint "Resistor_SMD:R_0402_1005Metric")
+    )
     (path "/a74c9d3b-864a-43d5-bde6-cbf00bb39165/b7ebb9f2-f07e-4a37-9537-24cd3b8b28c7"
       (reference "U?") (unit 4) (value "RV1126") (footprint "berryflight: RV1126")
@@
       (reference "Y?") (unit 1) (value "24Mhz") (footprint "")
     )
-    (path "/e25c5f3e-57b5-4d7a-a8af-98b1826cae36/210a6a86-46c6-44af-97eb-10f8190287ac"
-      (reference "U?") (unit 3) (value "RK809") (footprint "berryflight:QFN-68_EP_7x7_Pitch0.35mm")
-    )
-  )
+    (path "/2b4337a7-31ba-4b62-90e4-5bec465ff16f/210a6a86-46c6-44af-97eb-10f8190287ac"
+      (reference "U?") (unit 1) (value "RK809") (footprint "berryflight:QFN-68_EP_7x7_Pitch0.35mm")
+    )
+  )
