File: Hardware/core/pwr.kicad_sch (KiCad schematic)
At the start: 95 parts, among them U201 RV1126, U202 RK809

Commit message: moooaaarr power
Other:
- note added: "FB loop"
Changed lines of the file:
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@@
     )
+  )
+  (text "FB loop" (at 223.52 80.01 180)
+    (effects (font (size 1.27 1.27)) (justify right bottom))
+  )
+  (text "FB loop" (at 224.79 53.34 180)
+    (effects (font (size 1.27 1.27)) (justify right bottom))
   )
   (global_label "BC_VDD_VEPU" (shape input) (at 144.78 201.93 0) (fields_autoplaced)

Commit message: no ram yet
Parts:
- U1: renamed from U201; footprint berryflight: RV1126 -> berryflight:RV1126
- gave numbers to parts that had none: 44
- renumbered C201 to C1, C210 to C10, C211 to C11, C212 to C12, C213 to C13, C214 to C14, C215 to C15, C216 to C16, C217 to C17, C218 to C18, C219 to C19, C202 to C2, C220 to C20, C221 to C21, C223 to C22, C224 to C23, C225 to C24, C222 to C25, C226 to C26, C227 to C27, C229 to C28, C230 to C29, C203 to C3, C231 to C30, C232 to C31, C233 to C32, C234 to C33, C235 to C34, C204 to C4, C205 to C5, C206 to C6, C207 to C7, C208 to C8, C209 to C9, L201 to L1, L202 to L2, L203 to L3, L204 to L4, R201 to R1, R211 to R10, R202 to R2, R203 to R3, R204 to R4, R206 to R5, R207 to R6, R208 to R7, R209 to R8, R210 to R9, U202 to U2
