File: Hardware/core/byte0.kicad_pcb (KiCad board)
At the start: 6 copper layers, 37 x 37 mm, 185 parts, among them U1 RV1126, U2 RK809, U3 NCEPNA6M4-0808, U4 SY8089AAAC, U5 SY8089AAAC, U6 SY8113B, U7 SGM2203-5.0, Y1 24Mhz

Commit message: byte1 and 2
Connections:
- U1 pad A2: /Storage and RAM/DQ16 -> /Storage and RAM/DQ24
- U1 pad A3: /Storage and RAM/DQ17 -> /Storage and RAM/DQ25
- U1 pad B1: /Storage and RAM/DQ22 -> /Storage and RAM/DQ30
- U1 pad B2: /Storage and RAM/DQ23 -> /Storage and RAM/DQ31
- U1 pad B3: /Storage and RAM/DM2 -> /Storage and RAM/DM3
- U1 pad D3: /Storage and RAM/DQS2P -> /Storage and RAM/DQS3P
- U1 pad E3: /Storage and RAM/DQS2N -> /Storage and RAM/DQS3N
- U1 pad F4: /Storage and RAM/DQ19 -> /Storage and RAM/DQ27
- U1 pad G3: /Storage and RAM/DQ21 -> /Storage and RAM/DQ29
- U1 pad G4: /Storage and RAM/DQ18 -> /Storage and RAM/DQ26
- U1 pad H3: /Storage and RAM/DQ20 -> /Storage and RAM/DQ28
- U1 pad J1: /Storage and RAM/DQ26 -> /Storage and RAM/DQ18
- U1 pad J2: /Storage and RAM/DQ27 -> /Storage and RAM/DQ19
- U1 pad K1: /Storage and RAM/DQ24 -> /Storage and RAM/DQ16
- U1 pad K2: /Storage and RAM/DQ25 -> /Storage and RAM/DQ17
- U1 pad L1: /Storage and RAM/DQ29 -> /Storage and RAM/DQ21
- U1 pad M1: /Storage and RAM/DQ30 -> /Storage and RAM/DQ22
- U1 pad M2: /Storage and RAM/DM3 -> /Storage and RAM/DM2
- U1 pad N1: /Storage and RAM/DQS3N -> /Storage and RAM/DQS2N
- U1 pad N2: /Storage and RAM/DQS3P -> /Storage and RAM/DQS2P
- U1 pad P1: /Storage and RAM/DQ31 -> /Storage and RAM/DQ23
- U1 pad P2: /Storage and RAM/DQ28 -> /Storage and RAM/DQ20
- U1 pad T1: /Storage and RAM/MMC_CLK -> /Storage and RAM/CLK
Routing:
- net /Storage and RAM/DQS1P: track 20.2 -> 0.00 mm
- net /Storage and RAM/DM3: track 19.6 -> 0.00 mm
- net /Storage and RAM/DQS1N: track 17.7 -> 0.00 mm
- net /Storage and RAM/DQS3N: track 15.5 -> 0.00 mm
- net /Storage and RAM/DQ8: track 13.7 -> 0.00 mm
- net /Storage and RAM/DM1: track 13.7 -> 0.00 mm
- net /Storage and RAM/MMC_CMD: track 13.0 -> 0.00 mm
- net /Storage and RAM/DQS3P: track 11.2 -> 0.00 mm
- net /Storage and RAM/MMC_D7: track 10.9 -> 0.00 mm
- net /Storage and RAM/MMC_D3: track 9.47 -> 0.00 mm
- net /Storage and RAM/MMC_D2: track 6.79 -> 0.00 mm
- net /Storage and RAM/MMC_D6: track 6.36 -> 0.00 mm
- net /Storage and RAM/MMC_D0: track 5.35 -> 0.00 mm
- net /Storage and RAM/DQ30: track 4.88 -> 0.00 mm
- net /Storage and RAM/DQ10: track 4.72 -> 0.00 mm
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