File: Hardware/core/memory.kicad_sch (KiCad schematic)
At the start: 0 parts

Commit message: eMCP
Parts:
- added U? (x5): NCEPNA6M4-0808, symbol berryflight:NCEPNA6M4-0808

Commit message: DDR
Parts:
- added U? (x2): RV1126, berryflight: RV1126, symbol berryflight:RV1126
Connections:
- net DQ21: now reaches U?.AA10 (DQ21)
- net DQ21: now also U?.L1 (DDR_DQ21)
- net DQ20: now reaches U?.AA12 (DQ20)
- net DQ20: now also U?.P2 (DDR_DQ20)
- net DQ19: now reaches U?.AA13 (DQ19)
- net DQ19: now also U?.J2 (DDR_DQ19)
- net DQ18: now reaches U?.AB10 (DQ18)
- net DQ18: now also U?.J1 (DDR_DQ18)
- net DQ17: now reaches U?.AB11 (DQ17)
- net DQ17: now also U?.K2 (DDR_DQ17)
- net DQ16: now reaches U?.AB12 (DQ16)
- net DQ16: now also U?.K1 (DDR_DQ16)
- net DQ29: now reaches U?.F10 (DQ29)
- net DQ29: now also U?.G3 (DDR_DQ29)
- net DQ30: now reaches U?.F11 (DQ30)
- net DQ30: now also U?.B1 (DDR_DQ30)
- net DQ31: now reaches U?.F12 (DQ31)
- net DQ31: now also U?.B2 (DDR_DQ31)
- net DQ26: now reaches U?.G10 (DQ26)
- net DQ26: now also U?.G4 (DDR_DQ26)
- net DQ27: now reaches U?.G12 (DQ27)
- net DQ27: now also U?.F4 (DDR_DQ27)
- net DQ28: now reaches U?.G13 (DQ28)
- net DQ28: now also U?.H3 (DDR_DQ28)
- net DQ24: now reaches U?.H11 (DQ24)
- net DQ24: now also U?.A2 (DDR_DQ24)
- net DQ25: now reaches U?.H13 (DQ25)
- net DQ25: now also U?.A3 (DDR_DQ25)
- net A9: now reaches U?.H2 (CA9)
- net A9: now also U?.B9 (DDR_A9)
- net DQS3N: now reaches U?.H9 (DQS3_t)
- net DQS3N: now also U?.E3 (DDR_DQS3N)
- net DM3: now reaches U?.J10 (DM3)
- net DM3: now also U?.B3 (DDR_DM3)
- net DQ15: now reaches U?.J12 (DQ15)
- net DQ15: now also U?.C2 (DDR_DQ15)
- net A8: now reaches U?.J2 (CA8)
- net A8: now also U?.A8 (DDR_A8)
- net A7: now reaches U?.J3 (CA7)
- net A7: now also U?.B8 (DDR_A7)
- net DQS3P: now reaches U?.J9 (DQS3_c)
- net DQS3P: now also U?.D3 (DDR_DQS3P)
- net DQ13: now reaches U?.K11 (DQ13)
- net DQ13: now also U?.E1 (DDR_DQ13)
- net DQ14: now reaches U?.K13 (DQ14)
- net DQ14: now also U?.C1 (DDR_DQ14)
- net A6: now reaches U?.K3 (CA6)
- net A6: now also U?.C8 (DDR_A6)
- net DQ12: now reaches U?.L11 (DQ12)
- net DQ12: now also U?.G1 (DDR_DQ12)
- net DQ11: now reaches U?.L13 (DQ11)
- net DQ11: now also U?.H1 (DDR_DQ11)
- net A5: now reaches U?.L3 (CA5)
- net A5: now also U?.A7 (DDR_A5)
- net DQ10: now reaches U?.M11 (DQ10)
- net DQ10: now also U?.H2 (DDR_DQ10)
- net DQ9: now reaches U?.M13 (DQ9)
- net DQ9: now also U?.D1 (DDR_DQ9)
- net DQS1N: now reaches U?.M9 (DQS1_t)
- net DQS1N: now also U?.F1 (DDR_DQS1N)
- net DM1: now reaches U?.N10 (DM1)
- net DM1: now also U?.E2 (DDR_DM1)
- net DQ8: now reaches U?.N12 (DQ8)
- net DQ8: now also U?.D2 (DDR_DQ8)
- net DQS1P: now reaches U?.N9 (DQS1_c)
- net DQS1P: now also U?.F2 (DDR_DQS1P)
- net DM0: now reaches U?.R10 (DM0)
- net DM0: now also U?.N3 (DDR_DM0)
- net DQ7: now reaches U?.R12 (DQ7)
- net DQ7: now also U?.P3 (DDR_DQ7)
- net DQS0P: now reaches U?.R9 (DQS0_c)
- net DQS0P: now also U?.L4 (DDR_DQS0P)
- net DQ5: now reaches U?.T11 (DQ5)
- net DQ5: now also U?.K3 (DDR_DQ5)
- net DQ6: now reaches U?.T13 (DQ6)
- net DQ6: now also U?.M4 (DDR_DQ6)
- net DQS0N: now reaches U?.T9 (DQS0_t)
- net DQS0N: now also U?.L3 (DDR_DQS0N)
- net DQ3: now reaches U?.U11 (DQ3)
- net DQ3: now also U?.N4 (DDR_DQ3)
- net DQ4: now reaches U?.U13 (DQ4)
- net DQ4: now also U?.J3 (DDR_DQ4)
- net DQ1: now reaches U?.V11 (DQ1)
- net DQ1: now also U?.J4 (DDR_DQ1)
- net DQ2: now reaches U?.V13 (DQ2)
- net DQ2: now also U?.P4 (DDR_DQ2)
- net A4: now reaches U?.V3 (CA4)
- net A4: now also U?.A9 (DDR_A4)
- net DM2: now reaches U?.W10 (DM2)
- net DM2: now also U?.M2 (DDR_DM2)
- net DQ0: now reaches U?.W12 (DQ0)
- net DQ0: now also U?.K4 (DDR_DQ0)
- net A2: now reaches U?.W2 (CA2)
- net A2: now also U?.B11 (DDR_A2)
- net A3: now reaches U?.W3 (CA3)
- net A3: now also U?.B6 (DDR_A3)
- net DQS2P: now reaches U?.W9 (DQS2_c)
- net DQS2P: now also U?.N2 (DDR_DQS2P)
- net DQ23: now reaches U?.Y11 (DQ23)
- net DQ23: now also U?.P1 (DDR_DQ23)
- net DQ22: now reaches U?.Y13 (DQ22)
- net DQ22: now also U?.M1 (DDR_DQ22)
- net A0: now reaches U?.Y2 (CA0)
- net A0: now also U?.C9 (DDR_A0)
- net A1: now reaches U?.Y3 (CA1)
- net A1: now also U?.B7 (DDR_A1)
- net DQS2N: now reaches U?.Y9 (DQS2_t)
- net DQS2N: now also U?.N1 (DDR_DQS2N)
- net ZQ: now reaches U?.G2 (ZQ)
- net ZQ: now also U?.E5 (DDR_RZQ)
- net CLKP: now reaches U?.N3 (CLK_c)
- net CLKP: now also U?.D4 (DDR_CLKP)
- net ODT: now reaches U?.P10 (ODT)
- net ODT: now also U?.A5 (DDR_ODT0)
- net CLKN: now reaches U?.P3 (CLK_t)
- net CLKN: now also U?.D5 (DDR_CLKN)
- net CKE: now reaches U?.T2 (CKE0)
- net CKE: now also U?.C6 (DDR_CKE)
- net CS1: now reaches U?.T3 (CS1_n)
- net CS0: now reaches U?.U3 (CS0_n)
- net CS0: now also U?.B4 (DDR_CS0N)
Other:
- moved on the sheet: U?A, U?B, U?C, U?D, U?E

Commit message: no ram yet
Parts:
- removed U?: RV1126, berryflight: RV1126, symbol berryflight:RV1126
- removed U? (x3): NCEPNA6M4-0808, symbol berryflight:NCEPNA6M4-0808
- added C89, C90, C91: 100nF, Capacitor_SMD:C_0201_0603Metric, symbol Device:C
- added C92, C93, C94: 1uF, Capacitor_SMD:C_0402_1005Metric, symbol Device:C
- added C95: 10uF, Capacitor_SMD:C_0603_1608Metric, symbol Device:C
- added R73: 240R, Resistor_SMD:R_0402_1005Metric, symbol Device:R
- added unit 5 of U1
- added unit 5 of U3
- added unit 1 of U3
- added unit 2 of U3
- U1: renamed from U?; footprint berryflight: RV1126 -> berryflight:RV1126
- U3: renamed from U?; footprint (none) -> berryflight:BGA-221
Connections:
- net A0: now also U1.D10 (DDR_A0)
- net A1: now also U1.A8 (DDR_A1)
- net A2: now also U1.D11 (DDR_A2)
- net A3: now also U1.C9 (DDR_A3)
- net A4: now also U1.B8 (DDR_A4)
- net A5: now also U1.B9 (DDR_A5)
- net A6: now also U1.A9 (DDR_A6)
- net A7: now also U1.C11 (DDR_A7)
- net A8: now also U1.A10 (DDR_A8)
- net A9: now also U1.B11 (DDR_A9)
- net CKE: now also U1.A4 (DDR_CKE)
- net CLKN: now also U3.N3 (CLK_c), U1.D5 (DDR_CLKN); no longer U3.P3 (CLK_t)
- net CLKP: now also U3.P3 (CLK_t), U1.D4 (DDR_CLKP); no longer U3.N3 (CLK_c)
- net CS0: now also U1.A5 (DDR_CS0n)
- net CS1: now also U1.E7 (DDR_CS1n)
- net DM0: now also U1.N3 (DDR_DM0)
- net DM1: now also U1.E2 (DDR_DM1)
- net DM2: now also U1.M2 (DDR_DM2)
- net DM3: now also U1.B3 (DDR_DM3)
- net DQ0: now also U1.K4 (DDR_D2)
- net DQ1: now also U1.J4 (DDR_D6)
- net DQ10: now also U1.H2 (DDR_D8)
- net DQ11: now also U1.H1 (DDR_D9)
- net DQ12: now also U1.G1 (DDR_D12)
- net DQ13: now also U1.E1 (DDR_D13)
- net DQ14: now also U1.C1 (DDR_D14)
- net DQ15: now also U1.C2 (DDR_D15)
- net DQ16: now also U1.K1 (DDR_D19)
- net DQ17: now also U1.K2 (DDR_D18)
- net DQ18: now also U1.J1 (DDR_D23)
- net DQ19: now also U1.J2 (DDR_D22)
- net DQ2: now also U1.P4 (DDR_D4)
- net DQ20: now also U1.P2 (DDR_D21)
- net DQ21: now also U1.L1 (DDR_D16)
- net DQ22: now also U1.M1 (DDR_D17)
- net DQ23: now also U1.P1 (DDR_D20)
- net DQ24: now also U1.A2 (DDR_D30)
- net DQ25: now also U1.A3 (DDR_D31)
- net DQ26: now also U1.G4 (DDR_D28)
- net DQ27: now also U1.F4 (DDR_D29)
- net DQ28: now also U1.H3 (DDR_D24)
- net DQ29: now also U1.G3 (DDR_D25)
- net DQ3: now also U1.N4 (DDR_D0)
- net DQ30: now also U1.B1 (DDR_D26)
- net DQ31: now also U1.B2 (DDR_D27)
- net DQ4: now also U1.J3 (DDR_D3)
- net DQ5: now also U1.K3 (DDR_D7)
- net DQ6: now also U1.M4 (DDR_D5)
- net DQ7: now also U1.P3 (DDR_D1)
- net DQ8: now also U1.D2 (DDR_D10)
- net DQ9: now also U1.D1 (DDR_D11)
- net DQS0N: now also U3.R9 (DQS0_c), U1.L3 (DDR_DQS0N); no longer U3.T9 (DQS0_t)
- net DQS0P: now also U3.T9 (DQS0_t), U1.L4 (DDR_DQS0P); no longer U3.R9 (DQS0_c)
- net DQS1N: now also U3.N9 (DQS1_c), U1.F1 (DDR_DQS1N); no longer U3.M9 (DQS1_t)
- net DQS1P: now also U3.M9 (DQS1_t), U1.F2 (DDR_DQS1P); no longer U3.N9 (DQS1_c)
- net DQS2N: now also U3.W9 (DQS2_c), U1.N1 (DDR_DQS2N); no longer U3.Y9 (DQS2_t)
- net DQS2P: now also U3.Y9 (DQS2_t), U1.N2 (DDR_DQS2P); no longer U3.W9 (DQS2_c)
- net DQS3N: now also U3.J9 (DQS3_c), U1.E3 (DDR_DQS3N); no longer U3.H9 (DQS3_t)
- net DQS3P: now also U3.H9 (DQS3_t), U1.D3 (DDR_DQS3P); no longer U3.J9 (DQS3_c)
- net ODT: now also U1.B4 (DDR_ODT0)
- net MMC_RST: now reaches U1.R3 (FLASH_WPn/EMMC_RSTn/FSPI_CLK/GPIO1_A3_d)
- net MMC_RST: now also U3.C2 (RST)
- net CLK: now reaches U1.T1 (FLASH_CLE/EMMC_CLKO/GPIO0_D7_d)
- net MMC_CMD: now reaches U1.T4 (FLASH_WRn/EMMC_CMD/GPIO0_D5_u)
- net MMC_CMD: now also U3.A6 (CMD)
- net MMC_D7: now reaches U1.U3 (FLASH_D7/EMMC_D7/GPIO0_D3_u)
- net MMC_D7: now also U3.B4 (DAT7)
- net MMC_D6: now reaches U1.U4 (FLASH_D6/EMMC_D6/GPIO0_D2_u)
- net MMC_D6: now also U3.A5 (DAT6)
- net MMC_D5: now reaches U1.V1 (FLASH_D5/EMMC_D5/FSPI_CS1n/GPIO0_D1_u)
- net MMC_D5: now also U3.A10 (DAT5)
- net MMC_D4: now reaches U1.V2 (FLASH_D4/EMMC_D4/GPIO0_D0_u)
- net MMC_D4: now also U3.C9 (DAT4)
- net MMC_D3: now reaches U1.V3 (FLASH_D3/EMMC_D3/GPIO0_C7_u)
- net MMC_D3: now also U3.B5 (DAT3)
- net MMC_D2: now reaches U1.V4 (FLASH_D2/EMMC_D2/GPIO0_C6_u)
- net MMC_D2: now also U3.C6 (DAT2)
- net MMC_D1: now reaches U1.W1 (FLASH_D1/EMMC_D1/GPIO0_C5_u)
- net MMC_D1: now also U3.B10 (DAT1)
- net MMC_D0: now reaches U1.W2 (FLASH_D0/EMMC_D0/GPIO0_C4_u)
- net MMC_D0: now also U3.A9 (DAT0)
- new net: U3.A4 (VCCQ), U3.B6 (VCCQ), U3.B9 (VCCQ), U3.C11 (VCCQ), U3.C7 (VCCQ)
- new net: U3.B12 (VCC), U3.B13 (VCC), U3.B3 (VCC), U3.C4 (VCC), U3.D8 (VCC)
- new net: C89.1, C90.1, C91.1, C92.1, C93.1, C94.1, C95.1, U1.G7 (DDR_VDD), U1.G8 (DDR_VDD), U1.G9 (DDR_VDD), U1.H8 (DDR_VDD), U1.J7 (DDR_VDD), U1.K7 (DDR_VDD), U1.L7 (DDR_VDD)
- new net: U3.AA3 (VDD1), U3.AA5 (VDD1), U3.AB3 (VDD1), U3.AB4 (VDD1), U3.AB9 (VDD1), U3.F3 (VDD1), U3.F4 (VDD1), U3.F9 (VDD1), U3.G5 (VDD1)
- new net: U3.AA9 (VDDQ), U3.G9 (VDDQ), U3.H12 (VDDQ), U3.H8 (VDDQ), U3.J11 (VDDQ), U3.K10 (VDDQ), U3.K12 (VDDQ), U3.L8 (VDDQ), U3.L9 (VDDQ), U3.M10 (VDDQ), U3.M12 (VDDQ), U3.N11 (VDDQ), U3.R11 (VDDQ), U3.T10 (VDDQ), U3.T12 (VDDQ), U3.U8 (VDDQ), U3.U9 (VDDQ), U3.V10 (VDDQ), U3.V12 (VDDQ), U3.W11 (VDDQ), U3.Y12 (VDDQ), U3.Y8 (VDDQ)
- new net: U3.AB5 (VDD2), U3.AB8 (VDD2), U3.F5 (VDD2), U3.F8 (VDD2), U3.J5 (VDD2), U3.K5 (VDD2), U3.L2 (VDD2), U3.L5 (VDD2), U3.M5 (VDD2), U3.N5 (VDD2), U3.P11 (VDD2), U3.P5 (VDD2), U3.P8 (VDD2), U3.R5 (VDD2), U3.T5 (VDD2), U3.U5 (VDD2), U3.V5 (VDD2), U3.W5 (VDD2)
- new net: R73.1, U1.E5 (DDR_RZQ)
- new net GND: C89.2, C90.2, C91.2, C92.2, C93.2, C94.2, C95.2, R73.2, U1.F6 (DDR_AVSS), U3.A12 (VSSm), U3.A3 (VSSm), U3.A8 (VSSm), U3.AA11 (VSS), U3.AA2 (VSS), U3.AA4 (VSS), U3.AA8 (VSS), U3.B11 (VSSm), U3.B2 (VSSm), U3.B7 (VSSm), U3.C10 (VSSm), U3.C12 (VSSm), U3.C3 (VSSm), U3.C5 (VSSm), U3.C8 (VSSm), U3.D7 (VSSm), U3.F13 (VSS), U3.F2 (VSS), U3.G11 (VSS), U3.G4 (VSS), U3.G8 (VSS), U3.H10 (VSS), U3.H3 (VSS), U3.H4 (VSS), U3.H5 (VSS), U3.J13 (VSS), U3.J4 (VSS), U3.J8 (VSS), U3.K4 (VSS), U3.K8 (VSS), U3.K9 (VSS), U3.L10 (VSS), U3.L12 (VSS), U3.L4 (VSS), U3.M3 (VSS), U3.M4 (VSS), U3.M8 (VSS), U3.N13 (VSS), U3.N4 (VSS), U3.N8 (VSS), U3.P12 (VSS), U3.P2 (VSS), U3.P4 (VSS), U3.P9 (VSS), U3.R13 (VSS), U3.R3 (VSS), U3.R4 (VSS), U3.R8 (VSS), U3.T4 (VSS), U3.T8 (VSS), U3.U10 (VSS), U3.U12 (VSS), U3.U4 (VSS), U3.V4 (VSS), U3.V8 (VSS), U3.V9 (VSS), U3.W13 (VSS), U3.W4 (VSS), U3.W8 (VSS), U3.Y10 (VSS), U3.Y4 (VSS), U3.Y5 (VSS)
- new net MMC_CLK: U3.B8 (CLKm)
- new net VREF: U1.M6 (DDR_VREF)

Commit message: byte1 and 2
Connections:
- net CLK is gone; now on net MMC_CLK: U1.T1 (FLASH_CLE/EMMC_CLKO/GPIO0_D7_d)
- net CKE: no longer U3.T2 (CKE0)
- net CLKN: no longer U3.N3 (CLK_c)
- net CLKP: no longer U3.P3 (CLK_t)
- net CS0: no longer U3.U3 (CS0_n)
- net CS1: no longer U3.T3 (CS1_n)
- net DM2: now also U1.B3 (DDR_DM3); no longer U1.M2 (DDR_DM2)
- net DM3: now also U1.M2 (DDR_DM2); no longer U1.B3 (DDR_DM3)
- net DQ16: now also U1.A2 (DDR_D30); no longer U1.K1 (DDR_D19)
- net DQ17: now also U1.A3 (DDR_D31); no longer U1.K2 (DDR_D18)
- net DQ18: now also U1.G4 (DDR_D28); no longer U1.J1 (DDR_D23)
- net DQ19: now also U1.F4 (DDR_D29); no longer U1.J2 (DDR_D22)
- net DQ20: now also U1.H3 (DDR_D24); no longer U1.P2 (DDR_D21)
- net DQ21: now also U1.G3 (DDR_D25); no longer U1.L1 (DDR_D16)
- net DQ22: now also U1.B1 (DDR_D26); no longer U1.M1 (DDR_D17)
- net DQ23: now also U1.B2 (DDR_D27); no longer U1.P1 (DDR_D20)
- net DQ24: now also U1.K1 (DDR_D19); no longer U1.A2 (DDR_D30)
- net DQ25: now also U1.K2 (DDR_D18); no longer U1.A3 (DDR_D31)
- net DQ26: now also U1.J1 (DDR_D23); no longer U1.G4 (DDR_D28)
- net DQ27: now also U1.J2 (DDR_D22); no longer U1.F4 (DDR_D29)
- net DQ28: now also U1.P2 (DDR_D21); no longer U1.H3 (DDR_D24)
- net DQ29: now also U1.L1 (DDR_D16); no longer U1.G3 (DDR_D25)
- net DQ30: now also U1.M1 (DDR_D17); no longer U1.B1 (DDR_D26)
- net DQ31: now also U1.P1 (DDR_D20); no longer U1.B2 (DDR_D27)
- net DQS2N: now also U1.E3 (DDR_DQS3N); no longer U1.N1 (DDR_DQS2N)
- net DQS2P: now also U1.D3 (DDR_DQS3P); no longer U1.N2 (DDR_DQS2P)
- net DQS3N: now also U1.N1 (DDR_DQS2N); no longer U1.E3 (DDR_DQS3N)
- net DQS3P: now also U1.N2 (DDR_DQS2P); no longer U1.D3 (DDR_DQS3P)
- net ODT: no longer U3.P10 (ODT)
- net ZQ: no longer U3.G2 (ZQ)
Other:
- moved on the sheet: U3D
Changed lines of the file:
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@@
     (effects (font (size 1.27 1.27)) (justify right bottom))
   )
-  (label "DQ16" (at 31.75 97.79 180)
-    (effects (font (size 1.27 1.27)) (justify right bottom))
-  )
-  (label "DQ17" (at 31.75 100.33 180)
-    (effects (font (size 1.27 1.27)) (justify right bottom))
-  )
-  (label "DQ18" (at 31.75 102.87 180)
-    (effects (font (size 1.27 1.27)) (justify right bottom))
-  )
-  (label "DQ19" (at 31.75 105.41 180)
-    (effects (font (size 1.27 1.27)) (justify right bottom))
-  )
-  (label "DQ20" (at 31.75 107.95 180)
-    (effects (font (size 1.27 1.27)) (justify right bottom))
-  )
-  (label "DQ21" (at 31.75 110.49 180)
-    (effects (font (size 1.27 1.27)) (justify right bottom))
-  )
-  (label "DQ22" (at 31.75 113.03 180)
-    (effects (font (size 1.27 1.27)) (justify right bottom))
-  )
-  (label "DQ23" (at 31.75 115.57 180)
-    (effects (font (size 1.27 1.27)) (justify right bottom))
-  )
-  (label "DM2" (at 31.75 119.38 180)
-    (effects (font (size 1.27 1.27)) (justify right bottom))
-  )
-  (label "DQS2P" (at 31.75 123.19 180)
-    (effects (font (size 1.27 1.27)) (justify right bottom))
-  )
-  (label "DQS2N" (at 31.75 125.73 180)
-    (effects (font (size 1.27 1.27)) (justify right bottom))
-  )
-  (label "DQ24" (at 31.75 129.54 180)
-    (effects (font (size 1.27 1.27)) (justify right bottom))
-  )
-  (label "DQ25" (at 31.75 132.08 180)
-    (effects (font (size 1.27 1.27)) (justify right bottom))
-  )
-  (label "DQ26" (at 31.75 134.62 180)
-    (effects (font (size 1.27 1.27)) (justify right bottom))
-  )
-  (label "DQ27" (at 31.75 137.16 180)
-    (effects (font (size 1.27 1.27)) (justify right bottom))
-  )
-  (label "DQ28" (at 31.75 139.7 180)
-    (effects (font (size 1.27 1.27)) (justify right bottom))
-  )
-  (label "DQ29" (at 31.75 142.24 180)
-    (effects (font (size 1.27 1.27)) (justify right bottom))
-  )
-  (label "DQ30" (at 31.75 144.78 180)
-    (effects (font (size 1.27 1.27)) (justify right bottom))
-  )
-  (label "DQ31" (at 31.75 147.32 180)
-    (effects (font (size 1.27 1.27)) (justify right bottom))
-  )
-  (label "DM3" (at 31.75 151.13 180)
-    (effects (font (size 1.27 1.27)) (justify right bottom))
-  )
-  (label "DQS3P" (at 31.75 154.94 180)
-    (effects (font (size 1.27 1.27)) (justify right bottom))
-  )
-  (label "DQS3N" (at 31.75 157.48 180)
+  (label "DQ24" (at 31.75 97.79 180)
+    (effects (font (size 1.27 1.27)) (justify right bottom))
+  )
+  (label "DQ25" (at 31.75 100.33 180)
+    (effects (font (size 1.27 1.27)) (justify right bottom))
+  )
+  (label "DQ26" (at 31.75 102.87 180)
+    (effects (font (size 1.27 1.27)) (justify right bottom))
+  )
+  (label "DQ27" (at 31.75 105.41 180)
+    (effects (font (size 1.27 1.27)) (justify right bottom))
+  )
+  (label "DQ28" (at 31.75 107.95 180)
+    (effects (font (size 1.27 1.27)) (justify right bottom))
+  )
+  (label "DQ29" (at 31.75 110.49 180)
+    (effects (font (size 1.27 1.27)) (justify right bottom))
+  )
+  (label "DQ30" (at 31.75 113.03 180)
+    (effects (font (size 1.27 1.27)) (justify right bottom))
+  )
+  (label "DQ31" (at 31.75 115.57 180)
+    (effects (font (size 1.27 1.27)) (justify right bottom))
+  )
+  (label "DM3" (at 31.75 119.38 180)
+    (effects (font (size 1.27 1.27)) (justify right bottom))
+  )
+  (label "DQS3P" (at 31.75 123.19 180)
+    (effects (font (size 1.27 1.27)) (justify right bottom))
+  )
+  (label "DQS3N" (at 31.75 125.73 180)
+    (effects (font (size 1.27 1.27)) (justify right bottom))
+  )
+  (label "DQ16" (at 31.75 129.54 180)
+    (effects (font (size 1.27 1.27)) (justify right bottom))
+  )
+  (label "DQ17" (at 31.75 132.08 180)
+    (effects (font (size 1.27 1.27)) (justify right bottom))
+  )
+  (label "DQ18" (at 31.75 134.62 180)
+    (effects (font (size 1.27 1.27)) (justify right bottom))
+  )
+  (label "DQ19" (at 31.75 137.16 180)
+    (effects (font (size 1.27 1.27)) (justify right bottom))
+  )
+  (label "DQ20" (at 31.75 139.7 180)
+    (effects (font (size 1.27 1.27)) (justify right bottom))
+  )
+  (label "DQ21" (at 31.75 142.24 180)
+    (effects (font (size 1.27 1.27)) (justify right bottom))
+  )
+  (label "DQ22" (at 31.75 144.78 180)
+    (effects (font (size 1.27 1.27)) (justify right bottom))
+  )
+  (label "DQ23" (at 31.75 147.32 180)
+    (effects (font (size 1.27 1.27)) (justify right bottom))
+  )
+  (label "DM2" (at 31.75 151.13 180)
+    (effects (font (size 1.27 1.27)) (justify right bottom))
+  )
+  (label "DQS2P" (at 31.75 154.94 180)
+    (effects (font (size 1.27 1.27)) (justify right bottom))
+  )
+  (label "DQS2N" (at 31.75 157.48 180)
     (effects (font (size 1.27 1.27)) (justify right bottom))
   )
@@
     (effects (font (size 1.27 1.27)) (justify left bottom))
   )
-  (label "CLK" (at 298.704 64.516 0)
+  (label "MMC_CLK" (at 298.704 64.516 0)
     (effects (font (size 1.27 1.27)) (justify left bottom))
   )
@@
     (pin "2")
   )
-  (symbol (lib_id "berryflight:NCEPNA6M4-0808") (at 141.732 129.794 0) (unit 4)
-    (in_bom yes) (on_board yes)
-    (property "Reference" "U3" (id 0) (at 144.272 125.984 0))
-    (property "Value" "NCEPNA6M4-0808" (id 1) (at 144.272 128.524 0))
-    (property "Footprint" "berryflight:BGA-221" (id 2) (at 103.632 127.254 0)
-      (effects (font (size 1.27 1.27)) hide)
-    )
-    (property "Datasheet" "" (id 3) (at 103.632 127.254 0)
-      (effects (font (size 1.27 1.27)) hide)
-    )
+  (symbol (lib_id "berryflight:NCEPNA6M4-0808") (at 141.732 129.794 0) (mirror y) (unit 4)
+    (in_bom yes) (on_board yes)
+    (property "Reference" "U3" (id 0) (at 139.192 125.984 0))
+    (property "Value" "NCEPNA6M4-0808" (id 1) (at 139.192 128.524 0))
+    (property "Footprint" "berryflight:BGA-221" (id 2) (at 179.832 127.254 0)
+      (effects (font (size 1.27 1.27)) hide)
+    )
+    (property "Datasheet" "" (id 3) (at 179.832 127.254 0)
+      (effects (font (size 1.27 1.27)) hide)
+    )
